File: EGSE Board/_autosave-PowerSupplies.kicad_sch (KiCad schematic)
At the start: 30 parts, among them U1 VOR2121A8, U2 VOR2121A8, U3 INA238AQDGSRQ1, U4 INA238AQDGSRQ1, U5 INA238AQDGSRQ1, U7 ISO1540, U9 LD1117S33TR_SOT223

Commit message: EGSE board updates
Other:
- moved on the sheet: C10
Changed lines of the file:
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@@
+    (stroke (width 0) (type default))
+  )
+  (wire (pts (xy 226.06 86.36) (xy 226.06 87.63))
+    (stroke (width 0) (type default))
+  )
+  (wire (pts (xy 226.06 81.28) (xy 226.06 80.01))
     (stroke (width 0) (type default))
   )
@@
   )
   (wire (pts (xy 138.43 135.89) (xy 179.07 135.89))
-    (stroke (width 0) (type default))
-  )
-  (wire (pts (xy 226.06 85.09) (xy 226.06 87.63))
     (stroke (width 0) (type default))
   )
@@
     )
   )
-  (symbol (lib_id "Device:C_Small") (at 226.06 82.55 180) (unit 1)
-    (in_bom yes) (on_board yes) (dnp no) (fields_autoplaced)
-    (property "Reference" "C10" (at 228.6 81.2736 0)
+  (symbol (lib_id "Device:C_Small") (at 226.06 83.82 180) (unit 1)
+    (in_bom yes) (on_board yes) (dnp no) (fields_autoplaced)
+    (property "Reference" "C10" (at 228.6 82.5436 0)
       (effects (font (size 1.27 1.27)) (justify right))
     )
-    (property "Value" "100nF" (at 228.6 83.8136 0)
+    (property "Value" "100nF" (at 228.6 85.0836 0)
       (effects (font (size 1.27 1.27)) (justify right))
     )
-    (property "Footprint" "" (at 226.06 82.55 0)
-      (effects (font (size 1.27 1.27)) hide)
-    )
-    (property "Datasheet" "~" (at 226.06 82.55 0)
-      (effects (font (size 1.27 1.27)) hide)
-    )
+    (property "Footprint" "" (at 226.06 83.82 0)
+      (effects (font (size 1.27 1.27)) hide)
+    )
+    (property "Datasheet" "~" (at 226.06 83.82 0)
+      (effects (font (size 1.27 1.27)) hide)
+    )
