File: EGSE Board/HeaterSupply.kicad_sch (KiCad schematic)
At the start: 19 parts, among them Q1 2N2219, U10 OP227, U11 DAC121S101, U3 INA238AQDGSRQ1, U6 ISU0205S15, U8 MAX31865xAP, U9 LD1117S33TR_SOT223

Commit message: Change to heater power
Parts:
- removed C13, C14, C15 (x2): 0.1u, symbol Device:C_Small
- removed C3: 100nF, symbol Device:C_Small
- removed C9: 10nF, symbol Device:C_Small
- removed Q1: 2N2219, Package_TO_SOT_THT:TO-39-3, symbol Transistor_BJT:2N2219
- removed R1: 0.1R, symbol Device:R
- removed R17: 2k7, symbol Device:R
- removed R17: 4K, symbol Device:R
- removed U10: OP227, Package_DIP:DIP-14_W7.62mm, symbol UserLibrary:OP227GN
- removed U3: INA238AQDGSRQ1, Package_SO:VSSOP-10_3x3mm_P0.5mm, symbol Power_Management:INA238AQDGSRQ1
- removed U8: MAX31865xAP, Package_SO:SSOP-20_5.3x7.2mm_P0.65mm, symbol Sensor_Temperature:MAX31865xAP
- added R17: R, symbol Device:R
- added U8: OPA551P, Package_DIP:DIP-8_W7.62mm, symbol Amplifier_Operational:OPA551P
- R18: value 1k -> R
Connections:
- net -12V_Unswitched: now also U8.4 (V-)
- net GND: now also R17.2; no longer R18.2
- net at R18.1: now also R17.1, U8.2 (-)
- net at U11.1 (Va): now also U8.3 (+)
- net at C15.1, U6.8 (+VOUT): now also U8.7 (V+)
- new net: R18.2, U8.6
Other:
- note removed: "Current monitor for heater"
- note removed: "SPI interface for RTD"
- note removed: "unused OP227A in package"

Commit message: Friday updates. PCB first draft
Parts:
- C15: footprint (none) -> Capacitor_SMD:C_0402_1005Metric
- R17: value R -> 1k; footprint (none) -> Resistor_SMD:R_0612_1632Metric
- R18: value R -> 3k3; footprint (none) -> Resistor_SMD:R_0612_1632Metric
- U11: footprint SOT23-6 -> Package_TO_SOT_SMD:SOT-23-6
Connections:
- net +12V_HTR: now reaches R18.2, U8.6
- net +15V: now reaches C15.1, U6.8 (+VOUT), U8.7 (V+)
Other:
- moved on the sheet: C15, U11B, U9
Changed lines of the file:
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@@
 (kicad_sch (version 20230121) (generator eeschema)
   (paper "A4")
-  (junction (at 116.84 186.69) (diameter 0) (color 0 0 0 0)
-  )
-  (junction (at 109.22 186.69) (diameter 0) (color 0 0 0 0)
+  (junction (at 186.69 88.9) (diameter 0) (color 0 0 0 0)
+  )
+  (junction (at 179.07 88.9) (diameter 0) (color 0 0 0 0)
   )
   (junction (at 62.23 60.96) (diameter 0) (color 0 0 0 0)
   )
-  (junction (at 109.22 154.94) (diameter 0) (color 0 0 0 0)
+  (junction (at 179.07 57.15) (diameter 0) (color 0 0 0 0)
+  )
+  (junction (at 123.19 77.47) (diameter 0) (color 0 0 0 0)
   )
   (junction (at 72.39 43.18) (diameter 0) (color 0 0 0 0)
@@
   (junction (at 99.06 91.44) (diameter 0) (color 0 0 0 0)
   )
-  (junction (at 123.19 77.47) (diameter 0) (color 0 0 0 0)
-  )
   (junction (at 34.29 53.34) (diameter 0) (color 0 0 0 0)
   )
@@
     (stroke (width 0) (type default))
   )
-  (wire (pts (xy 109.22 154.94) (xy 109.22 167.64))
+  (wire (pts (xy 179.07 57.15) (xy 179.07 69.85))
     (stroke (width 0) (type default))
   )
@@
     (stroke (width 0) (type default))
   )
-  (wire (pts (xy 109.22 154.94) (xy 116.84 154.94))
-    (stroke (width 0) (type default))
-  )
-  (wire (pts (xy 99.06 186.69) (xy 109.22 186.69))
-    (stroke (width 0) (type default))
-  )
-  (wire (pts (xy 123.19 77.47) (xy 200.66 77.47))
+  (wire (pts (xy 179.07 57.15) (xy 186.69 57.15))
+    (stroke (width 0) (type default))
+  )
+  (wire (pts (xy 168.91 88.9) (xy 179.07 88.9))
+    (stroke (width 0) (type default))
+  )
+  (wire (pts (xy 123.19 77.47) (xy 128.27 77.47))
     (stroke (width 0) (type default))
   )
@@
     (stroke (width 0) (type default))
   )
-  (wire (pts (xy 99.06 162.56) (xy 99.06 186.69))
-    (stroke (width 0) (type default))
-  )
-  (wire (pts (xy 116.84 187.96) (xy 116.84 186.69))
-    (stroke (width 0) (type default))
-  )
-  (wire (pts (xy 116.84 186.69) (xy 116.84 185.42))
+  (wire (pts (xy 168.91 64.77) (xy 168.91 88.9))
+    (stroke (width 0) (type default))
+  )
+  (wire (pts (xy 186.69 90.17) (xy 186.69 88.9))
+    (stroke (width 0) (type default))
+  )
+  (wire (pts (xy 186.69 88.9) (xy 186.69 87.63))
     (stroke (width 0) (type default))
   )
@@
     (stroke (width 0) (type default))
   )
-  (wire (pts (xy 106.68 154.94) (xy 109.22 154.94))
+  (wire (pts (xy 176.53 57.15) (xy 179.07 57.15))
     (stroke (width 0) (type default))
   )
@@
     (stroke (width 0) (type default))
   )
-  (wire (pts (xy 109.22 186.69) (xy 116.84 186.69))
+  (wire (pts (xy 179.07 88.9) (xy 186.69 88.9))
     (stroke (width 0) (type default))
   )
@@
     (stroke (width 0) (type default))
   )
-  (wire (pts (xy 109.22 172.72) (xy 109.22 186.69))
+  (wire (pts (xy 179.07 74.93) (xy 179.07 88.9))
     (stroke (width 0) (type default))
   )
@@
   )
   (text "DAC driven from 3v3 supply\nresistor chosen such that 3.3v on\nDAC output gives 12.15V at output\n300R heater resistors give 40.5mA"
-    (at 62.23 109.22 0)
+    (at 83.82 96.52 0)
     (effects (font (size 1.27 1.27)) (justify right bottom))
+  )
+  (label "+15V" (at 87.63 43.18 0) (fields_autoplaced)
+    (effects (font (size 1.27 1.27)) (justify left bottom))
   )
   (global_label "GND" (shape input) (at 30.48 53.34 180) (fields_autoplaced)
@@
     (effects (font (size 1.27 1.27)) (justify right))
   )
-  (hierarchical_label "+5V" (shape input) (at 91.44 154.94 180) (fields_autoplaced)
+  (hierarchical_label "+12V_HTR" (shape output) (at 128.27 77.47 0) (fields_autoplaced)
+    (effects (font (size 1.27 1.27)) (justify left))
+  )
+  (hierarchical_label "+5V" (shape input) (at 161.29 57.15 180) (fields_autoplaced)
     (effects (font (size 1.27 1.27)) (justify right))
   )
@@
     )
   )
-  (symbol (lib_id "User_Library:DAC121S101") (at 116.84 172.72 0) (unit 2)
-    (in_bom yes) (on_board yes) (dnp no) (fields_autoplaced)
-    (property "Reference" "U11" (at 118.11 168.91 0)
-      (effects (font (size 1.27 1.27)) (justify left))
-    )
-    (property "Value" "DAC121S101" (at 118.11 171.45 0)
-      (effects (font (size 1.27 1.27)) (justify left))
-    )
-    (property "Footprint" "SOT23-6" (at 116.84 172.72 0)
+  (symbol (lib_id "User_Library:DAC121S101") (at 186.69 74.93 0) (unit 2)
+    (in_bom yes) (on_board yes) (dnp no) (fields_autoplaced)
+    (property "Reference" "U11" (at 187.96 71.12 0)
+      (effects (font (size 1.27 1.27)) (justify left))
+    )
+    (property "Value" "DAC121S101" (at 187.96 73.66 0)
+      (effects (font (size 1.27 1.27)) (justify left))
+    )
+    (property "Footprint" "Package_TO_SOT_SMD:SOT-23-6" (at 186.69 74.93 0)
       (effects (font (size 1.27 1.27)) (justify bottom) hide)
     )
-    (property "Datasheet" "" (at 116.84 172.72 0)
+    (property "Datasheet" "" (at 186.69 74.93 0)
       (effects (font (size 1.27 1.27)) hide)
     )
@@
       (effects (font (size 1.27 1.27)))
     )
-    (property "Footprint" "SOT23-6" (at 55.88 77.47 0)
+    (property "Footprint" "Package_TO_SOT_SMD:SOT-23-6" (at 55.88 77.47 0)
       (effects (font (size 1.27 1.27)) (justify bottom) hide)
     )
@@
       (effects (font (size 1.27 1.27)))
     )
-    (property "Value" "R" (at 111.76 87.63 90)
-      (effects (font (size 1.27 1.27)))
-    )
-    (property "Footprint" "" (at 111.76 93.218 90)
+    (property "Value" "3k3" (at 111.76 87.63 90)
+      (effects (font (size 1.27 1.27)))
+    )
+    (property "Footprint" "Resistor_SMD:R_0612_1632Metric" (at 111.76 93.218 90)
       (effects (font (size 1.27 1.27)) hide)
     )
@@
     )
   )
-  (symbol (lib_id "Regulator_Linear:LD1117S33TR_SOT223") (at 99.06 154.94 0) (unit 1)
-    (in_bom yes) (on_board yes) (dnp no) (fields_autoplaced)
-    (property "Reference" "U9" (at 99.06 148.59 0)
-      (effects (font (size 1.27 1.27)))
-    )
-    (property "Value" "LD1117S33TR_SOT223" (at 99.06 151.13 0)
-      (effects (font (size 1.27 1.27)))
-    )
-    (property "Footprint" "Package_TO_SOT_SMD:SOT-223-3_TabPin2" (at 99.06 149.86 0)
-      (effects (font (size 1.27 1.27)) hide)
-    )
-    (property "Datasheet" "http://www.st.com/st-web-ui/static/active/en/resource/technical/document/datasheet/CD00000544.pdf" (at 101.6 161.29 0)
+  (symbol (lib_id "Regulator_Linear:LD1117S33TR_SOT223") (at 168.91 57.15 0) (unit 1)
+    (in_bom yes) (on_board yes) (dnp no) (fields_autoplaced)
+    (property "Reference" "U9" (at 168.91 50.8 0)
+      (effects (font (size 1.27 1.27)))
+    )
+    (property "Value" "LD1117S33TR_SOT223" (at 168.91 53.34 0)
+      (effects (font (size 1.27 1.27)))
+    )
+    (property "Footprint" "Package_TO_SOT_SMD:SOT-223-3_TabPin2" (at 168.91 52.07 0)
+      (effects (font (size 1.27 1.27)) hide)
+    )
+    (property "Datasheet" "http://www.st.com/st-web-ui/static/active/en/resource/technical/document/datasheet/CD00000544.pdf" (at 171.45 63.5 0)
       (effects (font (size 1.27 1.27)) hide)
     )
@@
     )
   )
-  (symbol (lib_id "power:GND") (at 116.84 187.96 0) (unit 1)
-    (in_bom yes) (on_board yes) (dnp no) (fields_autoplaced)
-    (property "Reference" "#PWR029" (at 116.84 194.31 0)
-      (effects (font (size 1.27 1.27)) hide)
-    )
-    (property "Value" "GND" (at 116.84 193.04 0)
-      (effects (font (size 1.27 1.27)))
-    )
-    (property "Footprint" "" (at 116.84 187.96 0)
-      (effects (font (size 1.27 1.27)) hide)
-    )
-    (property "Datasheet" "" (at 116.84 187.96 0)
+  (symbol (lib_id "power:GND") (at 186.69 90.17 0) (unit 1)
+    (in_bom yes) (on_board yes) (dnp no) (fields_autoplaced)
+    (property "Reference" "#PWR029" (at 186.69 96.52 0)
+      (effects (font (size 1.27 1.27)) hide)
+    )
+    (property "Value" "GND" (at 186.69 95.25 0)
+      (effects (font (size 1.27 1.27)))
+    )
+    (property "Footprint" "" (at 186.69 90.17 0)
+      (effects (font (size 1.27 1.27)) hide)
+    )
+    (property "Datasheet" "" (at 186.69 90.17 0)
       (effects (font (size 1.27 1.27)) hide)
     )
@@
     )
   )
-  (symbol (lib_id "Device:C_Small") (at 109.22 170.18 0) (unit 1)
-    (in_bom yes) (on_board yes) (dnp no) (fields_autoplaced)
-    (property "Reference" "C15" (at 111.76 168.9163 0)
-      (effects (font (size 1.27 1.27)) (justify left))
-    )
-    (property "Value" "0.1u" (at 111.76 171.4563 0)
-      (effects (font (size 1.27 1.27)) (justify left))
-    )
-    (property "Footprint" "" (at 109.22 170.18 0)
-      (effects (font (size 1.27 1.27)) hide)
-    )
-    (property "Datasheet" "~" (at 109.22 170.18 0)
+  (symbol (lib_id "Device:C_Small") (at 179.07 72.39 0) (unit 1)
+    (in_bom yes) (on_board yes) (dnp no) (fields_autoplaced)
+    (property "Reference" "C15" (at 181.61 71.1263 0)
+      (effects (font (size 1.27 1.27)) (justify left))
+    )
+    (property "Value" "0.1u" (at 181.61 73.6663 0)
+      (effects (font (size 1.27 1.27)) (justify left))
+    )
+    (property "Footprint" "Capacitor_SMD:C_0402_1005Metric" (at 179.07 72.39 0)
+      (effects (font (size 1.27 1.27)) hide)
+    )
+    (property "Datasheet" "~" (at 179.07 72.39 0)
       (effects (font (size 1.27 1.27)) hide)
     )
@@
       (effects (font (size 1.27 1.27)) (justify left))
     )
-    (property "Value" "R" (at 96.52 99.06 0)
-      (effects (font (size 1.27 1.27)) (justify left))
-    )
-    (property "Footprint" "" (at 92.202 97.79 90)
+    (property "Value" "1k" (at 96.52 99.06 0)
+      (effects (font (size 1.27 1.27)) (justify left))
+    )
+    (property "Footprint" "Resistor_SMD:R_0612_1632Metric" (at 92.202 97.79 90)
       (effects (font (size 1.27 1.27)) hide)
     )
@@
       (effects (font (size 1.27 1.27)) (justify left))
     )
-    (property "Footprint" "" (at 72.39 52.07 0)
-      (effects (font (size 1.27 1.27)) hide)
-    )
+    (property "Footprint" "Capacitor_SMD:C_0402_1005Metric" (at 72.39 52.07 0)
+      (effects (font (size 1.27 1.27)) hide)
+    )

Commit message: Regular update
Created Gerber files for production
Changed names in arduino code to reflect signal names used by MSSL and on EGSE board
Parts:
- R17, R18: footprint Resistor_SMD:R_0612_1632Metric -> Resistor_SMD:R_0805_2012Metric
Changed lines of the file:
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@@
       (effects (font (size 1.27 1.27)))
     )
-    (property "Footprint" "Resistor_SMD:R_0612_1632Metric" (at 111.76 93.218 90)
+    (property "Footprint" "Resistor_SMD:R_0805_2012Metric" (at 111.76 93.218 90)
       (effects (font (size 1.27 1.27)) hide)
     )
@@
       (effects (font (size 1.27 1.27)) (justify left))
     )
-    (property "Footprint" "Resistor_SMD:R_0612_1632Metric" (at 92.202 97.79 90)
+    (property "Footprint" "Resistor_SMD:R_0805_2012Metric" (at 92.202 97.79 90)
       (effects (font (size 1.27 1.27)) hide)
     )

Commit message: Updated
Other:
- note added: "DAC driven from 3v3 supply resistor chosen such that 3.3v on DAC output gives 12.15V at output 300R heater resistors give 40.5mA (0.55W)"
- note removed: "DAC driven from 3v3 supply resistor chosen such that 3.3v on DAC output gives 12.15V at output 300R heater resistors give 40.5mA"
Changed lines of the file:
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@@
     (effects (font (size 2.54 2.54)) (justify right bottom))
   )
-  (text "DAC driven from 3v3 supply\nresistor chosen such that 3.3v on\nDAC output gives 12.15V at output\n300R heater resistors give 40.5mA"
+  (text "DAC driven from 3v3 supply\nresistor chosen such that 3.3v on\nDAC output gives 12.15V at output\n300R heater resistors give 40.5mA (0.55W)\n"
     (at 83.82 96.52 0)
     (effects (font (size 1.27 1.27)) (justify right bottom))
